File: Hardware/Sensor_Nodes_V2/gr25_nodes.kicad_pcb (KiCad board)
At the start: 4 copper layers, 32 x 48.8 mm, 48 parts, among them J1 SWD, J2 IO1, J3 I02, J4 PWR, U1 SN65HVD230, U2 AP63205WU, U3 AMS1117-3.3, U4 STM32F103C8Tx, Y1 16MHz

Commit message: some chnages, for tracking purpose
Parts:
- removed C1, C10, C11, C13, C14, C2, C6, C7: 100nF, Capacitor_SMD:C_0603_1608Metric
- removed C12, C8, C9: 4.7uF, Capacitor_SMD:C_0603_1608Metric
- removed C15: 10uF, Capacitor_SMD:C_0603_1608Metric
- removed C16, C4, C5: 22uF, Capacitor_SMD:C_1206_3216Metric
- removed C17, C19: 10pF, Capacitor_SMD:C_0603_1608Metric
- removed C3: 10uF, Capacitor_SMD:C_0805_2012Metric
- removed D1: 1N5819, Diode_SMD:D_SOD-323_HandSoldering
- removed D2, D3, D4, D5, D6: LED, Diode_SMD:D_0603_1608Metric
- removed FB1: 100R, Inductor_SMD:L_0805_2012Metric
- removed J1: SWD, Connector_PinHeader_2.54mm:PinHeader_1x04_P2.54mm_Vertical
- removed J2: IO1, Connector_PinHeader_2.54mm:PinHeader_1x18_P2.54mm_Vertical
- removed J3: I02, Connector_PinHeader_2.54mm:PinHeader_1x18_P2.54mm_Vertical
- removed J4: PWR, Connector_PinHeader_2.54mm:PinHeader_1x03_P2.54mm_Vertical
- removed JP1: 3.3V, Jumper:SolderJumper-2_P1.3mm_Bridged_RoundedPad1.0x1.5mm
- removed JP2: 5V, Jumper:SolderJumper-2_P1.3mm_Open_RoundedPad1.0x1.5mm
- removed JP3: +5vS, Jumper:SolderJumper-2_P1.3mm_Open_RoundedPad1.0x1.5mm
- removed JP4: Enable if VIO, Jumper:SolderJumper-2_P1.3mm_Open_RoundedPad1.0x1.5mm
- removed JP5: +3.3A, Jumper:SolderJumper-2_P1.3mm_Open_RoundedPad1.0x1.5mm
- removed JP6: +3.3vS, Jumper:SolderJumper-2_P1.3mm_Open_RoundedPad1.0x1.5mm
- removed JP7: BOOT, Jumper:SolderJumper-2_P1.3mm_Open_RoundedPad1.0x1.5mm
- removed L1: 4.7u, Inductor_SMD:L_Bourns-SRN4018
- removed R1, R2, R4, R5, R6: 220, Resistor_SMD:R_0603_1608Metric
- removed R3: 10k, Resistor_SMD:R_0603_1608Metric
- removed U1: SN65HVD230, Package_SO:SOIC-8_3.9x4.9mm_P1.27mm
- removed U2: AP63205WU, Package_TO_SOT_SMD:TSOT-23-6
- removed U3: AMS1117-3.3, Package_TO_SOT_SMD:SOT-223-3_TabPin2
- removed U4: STM32F103C8Tx, Package_QFP:LQFP-48_7x7mm_P0.5mm
- removed Y1: 16MHz, Crystal:Crystal_SMD_3225-4Pin_3.2x2.5mm
Routing:
- net GND: track 87.1 -> 0.00 mm, vias 36 -> 0
- net PA1: track 40.2 -> 0.00 mm
- net +3.3V: track 39.8 -> 0.00 mm, vias 14 -> 0
- net PA0: track 38.9 -> 0.00 mm
- net +5V: track 37.7 -> 0.00 mm
- net PA2: track 33.4 -> 0.00 mm
- net PB0: track 32.4 -> 0.00 mm, vias 1 -> 0
- net PB1: track 31.3 -> 0.00 mm, vias 1 -> 0
- net PB2: track 30.4 -> 0.00 mm, vias 1 -> 0
- net PB12: track 26.0 -> 0.00 mm, vias 1 -> 0
- net PB11: track 24.6 -> 0.00 mm, vias 1 -> 0
- net PB9: track 24.6 -> 0.00 mm, vias 1 -> 0
- net PB10: track 23.0 -> 0.00 mm, vias 1 -> 0
- net Net-(D2-A): track 22.1 -> 0.00 mm
- net PB8: track 21.5 -> 0.00 mm, vias 1 -> 0
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- removed copper zone on F.Cu, net (none)
- removed copper zone on F.Cu, net /3.3BC
Other:
- board outline removed
- board text removed: "12V"
- board text removed: "3V3"
- board text removed: "5V"
- board text removed: "GND"
- board text removed: "GND CLK DIO 3V3"
- board text removed: "PA0 PA1 PA2 PA3 PA4 PA5 PA6 PA7 CANL CANH GND PB10 PB11 NC GND"
- board text removed: "PB9 PB8 PB7 PB6 PB5 PB4 PB3 PA15 PA10 PA9 PA8 PB15 PB14 PB13 PB12 PB2 PB1 PB0"
