File: Hardware/Sensor_Nodes_V2/gr25_nodes.kicad_sch (KiCad schematic)
At the start: 49 parts, among them J1 SWD, J2 IO1, J3 I02, J4 PWR, U1 SN65HVD230, U2 AP63205WU, U3 AMS1117-3.3, U4 STM32F103C8Tx, U5 CH340E, Y1 16MHz

Commit message: added uart abstraction in examples/Testing
Parts:
- removed U5: CH340E, Package_SO:MSOP-10_3x3mm_P0.5mm, symbol Interface_USB:CH340E
Changed lines of the file:
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@@
-    )
-  )
-  (symbol (lib_id "Interface_USB:CH340E") (at 148.59 139.7 0) (unit 1)
-    (in_bom yes) (on_board yes) (dnp no) (fields_autoplaced)
-    (property "Reference" "U5" (at 150.5459 154.94 0)
-      (effects (font (size 1.27 1.27)) (justify left))
-    )
-    (property "Value" "CH340E" (at 150.5459 157.48 0)
-      (effects (font (size 1.27 1.27)) (justify left))
-    )
-    (property "Footprint" "Package_SO:MSOP-10_3x3mm_P0.5mm" (at 149.86 153.67 0)
-      (effects (font (size 1.27 1.27)) (justify left) hide)
-    )
-    (property "Datasheet" "https://www.mpja.com/download/35227cpdata.pdf" (at 139.7 119.38 0)
-      (effects (font (size 1.27 1.27)) hide)
-    )
-    (pin "1")
-    (pin "10")
-    (pin "2")
-    (pin "3")
-    (pin "4")
-    (pin "5")
-    (pin "6")
-    (pin "7")
-    (pin "8")
-    (pin "9")
-    (instances
-      (project "gr25_nodes"
-        (path "/af439857-71bc-46da-b029-0b772706e165"
-          (reference "U5") (unit 1)
-        )
-      )
     )
   )

Commit message: some chnages, for tracking purpose
Parts:
- added J5: Micro_SD_Card, symbol Connector:Micro_SD_Card
Other:
- moved on the sheet: C10, C11, C12, C13, C14, C15, C16, C17, C19, C2, C3, C4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
