File: Hardware/Sensor_Nodes_V3/_autosave-Main_MCU.kicad_sch (KiCad schematic)
At the start: 21 parts, among them J6 Conn_01x27_Socket, J7 Conn_01x27_Socket, U1 STM32G474RBTx, U3 MCP2542FDxMF, U6 MCP2542FDxMF

Commit message: finished the thing, need to optimize bom a little bit. need to flip some of the components too
Parts:
- C22: LCSC C19666 -> C57112
- L2: LCSC C1034 -> C1049
Changed lines of the file:
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@@
 			)
 		)
-		(property "LCSC" "C19666"
+		(property "LCSC" " C57112"
 			(at 209.55 64.77 0)
 			(effects
@@
 			)
 		)
-		(property "LCSC" "C1034"
+		(property "LCSC" "C1049"
 			(at 204.47 59.69 90)
 			(effects
