File: Hardware/Sensor_Nodes_V3/Bootloader.kicad_sch (KiCad schematic)
At the start: 36 parts, among them J1 Conn_01x06_Socket, Q1 S9013, U1 STM32F103C8Tx, Y1 8MHz

Commit message: tcm can schematic done, only needs to be routed
Changed lines of the file:
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@@
 (kicad_sch
-	(version 20231120)
+	(version 20250114)
 	(generator "eeschema")
-	(generator_version "8.0")
+	(generator_version "9.0")
 	(paper "A4")
 	(junction
