File: Hardware/Sensor_Nodes_V3/production/gr25_nodes_panelized.kicad_pcb (KiCad board)
At the start: 4 copper layers, 22.4 x 70.5 mm, 73 parts, among them J1 Conn_01x06_Socket, J2 Conn_01x27_Socket, J3 Conn_01x27_Socket, Q1 S9013, U1 STM32F103C8Tx, U2 STM32G474RBTx, U3 MCP2542FDxMF, U4 MCP2542FDxMF, U5 AMS1117-3.3, U6 TPS563200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

Commit message: sync
Other:
- board size 22.4 x 70.5 mm -> 22.1 x 70 mm
Changed lines of the file:
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@@
 		(tags "connector JST PH side entry")
 		(property "Reference" "J1"
-			(at -0.000001 -2.9 0)
+			(at 5.1 3.9 0)
 			(layer "F.SilkS")
 			(effects
@@
 		)
 	)
-	(gr_arc
-		(start 130 27.5)
-		(mid 130.707107 27.792893)
-		(end 131 28.5)
-		(stroke
-			(width 0.1)
-			(type default)
-		)
-		(layer "Edge.Cuts")
-	)
 	(gr_line
-		(start 130 27.5)
-		(end 109.6 27.5)
-		(stroke
-			(width 0.1)
-			(type default)
-		)
-		(layer "Edge.Cuts")
-	)
-	(gr_arc
-		(start 131 97)
-		(mid 130.707107 97.707107)
-		(end 130 98)
+		(start 130.75 97.75)
+		(end 130.775 27.775)
 		(stroke
 			(width 0.1)
@@
 	)
 	(gr_line
-		(start 109.6 98)
-		(end 130 98)
-		(stroke
-			(width 0.1)
-			(type default)
-		)
-		(layer "Edge.Cuts")
-	)
-	(gr_arc
-		(start 109.6 98)
-		(mid 108.892893 97.707107)
-		(end 108.6 97)
+		(start 108.75 27.75)
+		(end 108.725 97.75)
 		(stroke
 			(width 0.1)
@@
 	)
 	(gr_line
-		(start 108.6 28.5)
-		(end 108.6 97)
+		(start 130.775 27.775)
+		(end 108.75 27.75)
 		(stroke
 			(width 0.1)
@@
 	)
 	(gr_line
-		(start 131 97)
-		(end 131 28.5)
-		(stroke
-			(width 0.1)
-			(type default)
-		)
-		(layer "Edge.Cuts")
-	)
-	(gr_arc
-		(start 108.6 28.5)
-		(mid 108.892893 27.792893)
-		(end 109.6 27.5)
+		(start 108.725 97.75)
+		(end 130.75 97.75)
 		(stroke
 			(width 0.1)
@@
 		(polygon
 			(pts
-				(xy 123 89.85) (xy 123 85.4) (xy 116.8 85.4) (xy 116.8 89.9)
+				(xy 123 89.25) (xy 122.9 85.5) (xy 116.7 85.5) (xy 116.8 89.3)
 			)
 		)
